File: Hardware/Electronics/Kineses Board/Kineses_Board/Kineses_Board.kicad_pcb (KiCad board)
At the start: 2 copper layers, 26 x 65.6 mm, 19 parts, among them J1 Barrel_Jack, J2 Thumb, J3 Index, J4 Middle, J5 Ring, J6 Pinky, J7 Wrist, J8 HC-05

Commit message: Finished routing
Parts:
- moved J8 21.8 mm to (137.0, 102.7), turned to 90 degrees
- moved C1 4.35 mm to (142.6, 98.2)
- moved J3 4.23 mm to (158.6, 109.1)
- moved J4 4.23 mm to (158.6, 105.4)
- moved J6 4.23 mm to (158.6, 112.9)
- moved J2 4.23 mm to (158.6, 116.6)
- moved J5 4.23 mm to (158.6, 101.6)
- moved LOGO2 4.19 mm to (149.4, 98.2)
- moved J1 1.60 mm to (141.3, 106.2)
- moved MH1 1.30 mm to (159.2, 95.9)
- moved MH2 0.76 mm to (159.2, 63.5)
Routing:
- net /Thumb: track 0.00 -> 61.6 mm
- net /Pinky: track 0.00 -> 54.4 mm
- net /Index: track 0.00 -> 47.7 mm
- net /Middle: track 0.00 -> 35.7 mm
- net /Ring: track 0.00 -> 28.4 mm
- net /Wrist: track 0.00 -> 27.4 mm
- net /TX: track 0.00 -> 24.4 mm
- net /RX: track 0.00 -> 23.3 mm
- net /+5V: track 0.00 -> 23.0 mm
- net /VIN: track 0.00 -> 10.9 mm
- net Net-(A1-Pad1): track 0.00 -> 3.98 mm
- added copper zone on F.Cu, net /GND
- added copper zone on B.Cu, net /VIN
Other:
- board size 26 x 65.6 mm -> 27.6 x 67.3 mm

Commit message: Routing finished
Parts:
- J1: value Barrel_Jack -> Power; footprint Connector_BarrelJack:BarrelJack_CUI_PJ-063AH_Horizontal -> Connector_PinHeader_2.54mm:PinHeader_1x02_P2.54mm_Horizontal
- moved J8 12.5 mm to (149.5, 103.0), turned to 270 degrees
- moved J1 1.32 mm to (142.0, 107.3), turned to 270 degrees
Routing:
- net /TX: track 24.4 -> 16.9 mm
- net /RX: track 23.3 -> 17.1 mm
- net /+5V: track 23.0 -> 21.1 mm
Other:
- board text added: "+6V"
- board text added: "GND"

Commit message: Updated pics, added more to hardware section
Other:
- board text added: "UUID: 57560fb0-6e78-4d79-87aa -f23405300be4 BT ID: KINESIS_ARM"
Changed lines of the file:
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@@
   (general
     (thickness 1.6)
-    (drawings 27)
+    (drawings 28)
     (tracks 57)
     (zones 0)
@@
     )
   )
+  (gr_text "UUID: 57560fb0-6e78-4d79-87aa\n      -f23405300be4\nBT ID: KINESIS_ARM" (at 143.56 52.76 90) (layer B.SilkS)
+    (effects (font (size 1.5 1.5) (thickness 0.3)) (justify left mirror))
+  )
   (gr_text GND (at 145.28 108.06 90) (layer F.SilkS)

Commit message: Updated gerbers. Initial commit of interim Presentation
Parts:
- C1: footprint Capacitor_SMD:CP_Elec_4x4.5 -> Capacitor_SMD:CP_Elec_5x5.3
- moved C1 0.83 mm to (143.2, 98.7)
- moved J8 0.45 mm to (149.5, 103.5)
Routing:
- net /TX: track 16.9 -> 18.6 mm
Other:
- board text added: "+7V"
- board text removed: "+6V"
