File: Hardware/Electronics/Data Acquisition Board/ADC Breakout/DAQ Board.sch (KiCad schematic (older format))
At the start: 59 parts, among them J1 Conn_01x16, J2 Conn_01x16, U1 MCP1755T-5002E_SOT223-5, U2 LM3480-3.3

Commit message: Changed unused analog inputs to AVDD, removed mid supply voltage divider. Small routing change
Parts:
- removed R1, R2: 10k, Resistor_SMD:R_0603_1608Metric, symbol Device:R
Connections:
- net labels removed: MID_SUPPLY
- wire segments 261 -> 254
Other:
- note removed: "Mid-Supply Voltage Divider"
Changed lines of the file:
@@
 Connection ~ 3100 5600
 NoConn ~ 6500 5200
-$Comp
-L Device:R R?
-U 1 1 5E8AA917
-P 1450 6850
-AR Path="/5D7F9BD3/5E8AA917" Ref="R?"  Part="1"
-AR Path="/5E8AA917" Ref="R1"  Part="1"
-F 0 "R1" H 1520 6896 50  0000 L CNN
-F 1 "10k" H 1520 6805 50  0000 L CNN
-F 2 "Resistor_SMD:R_0603_1608Metric" V 1380 6850 50  0001 C CNN
-F 3 "~" H 1450 6850 50  0001 C CNN
-	1    1450 6850
-	1    0    0    -1
-$EndComp
-$Comp
-L Device:R R?
-U 1 1 5E8AA91E
-P 1450 7250
-AR Path="/5D7F9BD3/5E8AA91E" Ref="R?"  Part="1"
-AR Path="/5E8AA91E" Ref="R2"  Part="1"
-F 0 "R2" H 1520 7296 50  0000 L CNN
-F 1 "10k" H 1520 7205 50  0000 L CNN
-F 2 "Resistor_SMD:R_0603_1608Metric" V 1380 7250 50  0001 C CNN
-F 3 "~" H 1450 7250 50  0001 C CNN
-	1    1450 7250
-	1    0    0    -1
-$EndComp
-Wire Wire Line
-	1450 6500 1200 6500
-Wire Wire Line
-	1450 6500 1450 6700
-Wire Wire Line
-	1450 7000 1450 7050
-Wire Wire Line
-	1450 7050 1950 7050
-Connection ~ 1450 7050
-Wire Wire Line
-	1450 7050 1450 7100
-Wire Wire Line
-	1450 7400 1450 7550
-Wire Wire Line
-	1450 7550 1200 7550
-Text Label 1200 6500 0    50   ~ 0
-AVDD
-Text Label 1200 7550 0    50   ~ 0
-AVSS
-Text Label 1500 7050 0    50   ~ 0
-MID_SUPPLY
 Wire Wire Line
 	6100 3200 6000 3200
@@
 	6000 2950 5250 2950
 Connection ~ 6000 3200
-Text Label 5350 2950 0    50   ~ 0
-MID_SUPPLY
 $Comp
 L Device:C C?
@@
 Text Notes 8050 4950 0    50   ~ 0
 All GPIO Pins pulled to GND, unused
-Text Notes 650  6400 0    79   ~ 0
-Mid-Supply Voltage Divider
-Wire Notes Line
-	650  6300 2350 6300
-Wire Notes Line
-	2350 7700 650  7700
 Text Label 7800 5450 0    50   ~ 0
 ~RESET
@@
 Wire Wire Line
 	3400 2450 3400 2600
-Wire Notes Line
-	2350 6300 2350 7700
-Wire Notes Line
-	650  6300 650  7700
 Wire Wire Line
 	1950 3100 2700 3100
@@
 Text Label 7400 2250 0    50   ~ 0
 VCAP3
-Text Label 750  4950 0    50   ~ 0
-MID_SUPPLY
 Text Label 750  4750 0    50   ~ 0
 VREFP
@@
 Text Label 750  4200 0    50   ~ 0
 DVDD
+Text Label 5250 2950 0    50   ~ 0
+AVDD
 $EndSCHEMATC

Commit message: Removed pullup resistor on /CS. Reran production pdfs and plotted schematic
Parts:
- removed R16: 100k, Resistor_SMD:R_0603_1608Metric, symbol Device:R
Connections:
- net labels added: CLK
- wire segments 254 -> 251
- no-connect marks 8 -> 7
Other:
- note removed: "Pull-up CS\nto VDD for\nICP"
Changed lines of the file:
@@
 Text Label 8150 4550 0    50   ~ 0
 START
-NoConn ~ 8100 4450
 Text Label 8150 4350 0    50   ~ 0
 ~CS
@@
 Typical AVDD Rail\nsupply current 7.14mA.\nImax = 300mA
 $Comp
-L Device:R R?
-U 1 1 5E8AAB9B
-P 8850 4450
-AR Path="/5D7F9BD3/5E8AAB9B" Ref="R?"  Part="1"
-AR Path="/5E8AAB9B" Ref="R16"  Part="1"
-F 0 "R16" H 9000 4400 50  0000 C CNN
-F 1 "100k" H 9000 4500 50  0000 C CNN
-F 2 "Resistor_SMD:R_0603_1608Metric" V 8780 4450 50  0001 C CNN
-F 3 "~" H 8850 4450 50  0001 C CNN
-	1    8850 4450
-	1    0    0    -1
-$EndComp
-Wire Wire Line
-	8650 4350 8650 4600
-Wire Wire Line
-	8650 4600 8850 4600
-Wire Wire Line
-	8100 4350 8650 4350
-Connection ~ 8850 4600
-Wire Wire Line
-	8850 4600 9150 4600
-Wire Wire Line
-	8850 4300 9100 4300
-Text Label 8900 4300 0    50   ~ 0
-DVDD
-Text Notes 9150 4550 0    50   ~ 0
-Pull-up CS\nto VDD for\nICP
-$Comp
 L Connector_Generic:Conn_01x16 J?
 U 1 1 5E8AABAA
@@
 	1350 3200 750  3200
 Wire Wire Line
+	1350 3300 750  3300
+Wire Wire Line
 	1350 3400 750  3400
 Wire Wire Line
 	1350 3500 750  3500
 Wire Wire Line
+	1350 3700 750  3700
+Wire Wire Line
+	1350 3800 750  3800
+Wire Wire Line
+	1350 3900 750  3900
+Wire Wire Line
+	1350 4000 750  4000
+Wire Wire Line
+	1350 4100 750  4100
+Wire Wire Line
 	1350 3600 750  3600
 Wire Wire Line
-	1350 3700 750  3700
-Wire Wire Line
-	1350 3800 750  3800
-Wire Wire Line
-	1350 3900 750  3900
-Wire Wire Line
-	1350 4000 750  4000
-Wire Wire Line
-	1350 4100 750  4100
-Wire Wire Line
-	1350 3300 750  3300
-Wire Wire Line
 	1350 4200 750  4200
 Wire Wire Line
@@
 Wire Wire Line
 	1350 4950 750  4950
+Text Label 750  3300 0    50   ~ 0
+MOSI
 Text Label 750  3400 0    50   ~ 0
-MOSI
+~PWDN
 Text Label 750  3500 0    50   ~ 0
-~PWDN
-Text Label 750  3600 0    50   ~ 0
 ~RESET
 Text Label 750  3700 0    50   ~ 0
@@
 Text Label 5250 2950 0    50   ~ 0
 AVDD
+Text Label 750  3600 0    50   ~ 0
+CLK
+Wire Wire Line
+	8100 4450 8350 4450
+Text Label 8200 4450 0    50   ~ 0
+CLK
+Wire Wire Line
+	8100 4350 8350 4350
 $EndSCHEMATC
