File: Hardware/Electronics/Classification and Control Board/Classification and Contol Board.kicad_pcb (KiCad board)
At the start: 4 copper layers, 53.9 x 62.3 mm, 94 parts, among them J1 SWD Header, J10 USB_B_Mini, J2 Barrel_Jack, J3 Thumb, J4 Index, J5 Middle, J6 Ring, J7 Pinky, J8 Wrist, J9 HC05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

Commit message: CLASSIFICATION AND CONTROL BOARD PRODUCTION
Routing:
- net (no net): vias 1 -> 0
Other:
- board text added: "3V3"
- board text added: "GND"
- board text added: "NRST"
- board text added: "SWCLK"
- board text added: "SWDIO"
- board text added: "SWO"
Changed lines of the file:
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@@
   (general
     (thickness 1.6)
-    (drawings 16)
-    (tracks 729)
+    (drawings 22)
+    (tracks 728)
     (zones 0)
     (modules 94)
@@
       (effects (font (size 1 1) (thickness 0.15)))
     )
-    (fp_text value LTST-C171TGKT (at 0 1.43 90) (layer F.Fab)
+    (fp_text value LTST-C171TGKT (at -29.39 -0.59 90) (layer F.Fab)
       (effects (font (size 1 1) (thickness 0.15)))
     )
@@
       (effects (font (size 1 1) (thickness 0.15)))
     )
-    (fp_text value 6R (at 0 1.43 90) (layer F.Fab)
+    (fp_text value 6R (at 0.51 1.05 90) (layer F.Fab)
       (effects (font (size 1 1) (thickness 0.15)))
     )
@@
     (descr "Barrel Jack, 2.0mm ID, 5.5mm OD, 24V, 8A, no switch, https://www.cui.com/product/resource/pj-063ah.pdf")
     (tags "barrel jack cui dc power")
-    (fp_text reference J2 (at -6.89 4.75) (layer F.SilkS)
+    (fp_text reference J2 (at -3.86 13.52) (layer F.SilkS)
       (effects (font (size 1 1) (thickness 0.15)))
     )
@@
       (effects (font (size 1 1) (thickness 0.15)))
     )
-    (fp_text value 100n (at 0 1.43 270) (layer F.Fab)
+    (fp_text value 100n (at -0.04 1.19 270) (layer F.Fab)
       (effects (font (size 1 1) (thickness 0.15)))
     )
@@
     (descr "Through hole straight pin header, 1x06, 2.54mm pitch, single row")
     (tags "Through hole pin header THT 1x06 2.54mm single row")
-    (fp_text reference J1 (at 0.92 -2.79 90) (layer F.SilkS)
+    (fp_text reference J1 (at -2.44 1.8 180) (layer F.SilkS)
       (effects (font (size 1 1) (thickness 0.15)))
     )
@@
     (tags "usb micro receptacle")
     (attr smd)
-    (fp_text reference J10 (at -5.65 0.85 90) (layer F.SilkS)
+    (fp_text reference J10 (at -5.81 3.19 90) (layer F.SilkS)
       (effects (font (size 1 1) (thickness 0.15)))
     )
@@
     (tags diode)
     (attr smd)
-    (fp_text reference D6 (at 2.402 0.098 90) (layer F.SilkS)
+    (fp_text reference D6 (at -2.31 0.05 90) (layer F.SilkS)
       (effects (font (size 1 1) (thickness 0.15)))
     )
@@
       (effects (font (size 1 1) (thickness 0.15)))
     )
-    (fp_text value 68R (at -0.05 -1.55 270) (layer F.Fab)
+    (fp_text value 68R (at -0.02 -1.19 270) (layer F.Fab)
       (effects (font (size 1 1) (thickness 0.15)))
     )
@@
       (net 4 /STM32F407VGTx/3V3))
   )
+  (gr_text 3V3 (at 145.8 112.33) (layer F.SilkS)
+    (effects (font (size 1 1) (thickness 0.15)))
+  )
+  (gr_text SWCLK (at 139.03 115.881428 90) (layer F.SilkS)
+    (effects (font (size 1 1) (thickness 0.15)))
+  )
+  (gr_text GND (at 137.39 114.952857 90) (layer F.SilkS)
+    (effects (font (size 1 1) (thickness 0.15)))
+  )
+  (gr_text SWDIO (at 134.85 115.738571 90) (layer F.SilkS)
+    (effects (font (size 1 1) (thickness 0.15)))
+  )
+  (gr_text NRST (at 132.29 115.31 90) (layer F.SilkS)
+    (effects (font (size 1 1) (thickness 0.15)))
+  )
+  (gr_text SWO (at 129.73 115.000476 90) (layer F.SilkS)
+    (effects (font (size 1 1) (thickness 0.15)))
+  )
   (gr_circle (center 142.79 113.77) (end 142.92 113.85) (layer F.SilkS) (width 0.4))
-  (gr_line (start 124.44 103.48) (end 125.36 102.02) (layer F.Fab) (width 0.2))
+  (gr_line (start 124.44 103.48) (end 124.64 102.6) (layer F.Fab) (width 0.2))
   (gr_line (start 124.38 125.47) (end 124.44 103.48) (layer F.Fab) (width 0.2))
   (gr_line (start 117.97 105.42) (end 119.97 104.1) (layer F.Fab) (width 0.2))
   (gr_line (start 110.93 105.77) (end 117.97 105.42) (layer F.Fab) (width 0.2))
   (gr_line (start 140.4 75.53) (end 141.79 80.17) (layer F.Fab) (width 0.2))
-  (dimension 54.040008 (width 0.3) (layer Dwgs.User)
-    (gr_text "54.040 mm" (at 141.373814 57.945002 359.9681926) (layer Dwgs.User)
+  (dimension 54.040008 (width 0.3) (layer F.Fab)
+    (gr_text "54.040 mm" (at 141.373814 57.945002 359.9681926) (layer F.Fab)
       (effects (font (size 1.5 1.5) (thickness 0.3)))
     )
@@
     (arrow2b (pts (xy 114.352648 60.030002) (xy 115.479477 59.444207)))
   )
-  (dimension 62.380007 (width 0.3) (layer Dwgs.User)
-    (gr_text "62.380 mm" (at 172.08507 92.453424 89.97244512) (layer Dwgs.User)
+  (dimension 62.380007 (width 0.3) (layer F.Fab)
+    (gr_text "62.380 mm" (at 172.08507 92.453424 89.97244512) (layer F.Fab)
       (effects (font (size 1.5 1.5) (thickness 0.3)))
     )
@@
   (gr_arc (start 118.29 119.7) (end 114.43 119.7) (angle -90) (layer Edge.Cuts) (width 0.15))
   (gr_arc (start 118.3 65.17) (end 118.3 61.31) (angle -90) (layer Edge.Cuts) (width 0.15))
-  (via (at 116.18 109.65) (size 0.8) (drill 0.4) (layers F.Cu B.Cu) (net 0))
+  (via (at 116.18 109.65) (size 0.8) (drill 0.4) (layers F.Cu B.Cu) (net 1))
   (via (at 156.26 92.63) (size 0.8) (drill 0.4) (layers F.Cu B.Cu) (net 1))
   (via (at 116.78 63.58) (size 0.8) (drill 0.4) (layers F.Cu B.Cu) (net 1))
@@
   (via (at 120.18 66.83) (size 0.8) (drill 0.4) (layers F.Cu B.Cu) (net 1))
   (via (at 119.97 70.01) (size 0.8) (drill 0.4) (layers F.Cu B.Cu) (net 1))
-  (via (at 120.18 78.83) (size 0.8) (drill 0.4) (layers F.Cu B.Cu) (net 1))
   (via (at 122.62 87.54) (size 0.8) (drill 0.4) (layers F.Cu B.Cu) (net 1))
   (via (at 126.02 89.9) (size 0.8) (drill 0.4) (layers F.Cu B.Cu) (net 1))
